File: power-module.kicad_pcb (KiCad board)
At the start: 2 copper layers, 28.2 x 28 mm, 8 parts, among them J1 Conn_01x03, U1 LM2575-3.3BT

Commit message: Gerbers added
Other:
- board text added: "Rev A"
Changed lines of the file:
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@@
       (outputformat 1)
       (mirror false)
-      (drillshape 1)
+      (drillshape 0)
       (scaleselection 1)
-      (outputdirectory "")
+      (outputdirectory "gerbers/")
     )
   )
@@
     (effects (font (size 1 1) (thickness 0.15)) (justify mirror))
   )
+  (gr_text "Rev A" (at 157.15 85.85 90) (layer "F.SilkS")
+    (effects (font (size 1 1) (thickness 0.15)))
+  )
   (gr_text "Power Board 2575" (at 148.1 92.9) (layer "F.SilkS")
